File: Hardware/0. Project/PowerSpy.brd (EAGLE design)
At the start: 55 x 80 mm, 83 parts, among them IC1 CP2102N-A01-GQFN28, P1 Mini-Fit 4T, T1 SS8050, T2 SS8050, U1 NCP1117ST33T3G, U2 HLK-PM01, U3 ADS1115IDGST, U4 ESP32-WROOM-32D, X1 4T PJ-321, X2 4T PJ-321, X3 USB Micro B

Commit message: Schematic done. PCB layout almost done.
Parts:
- moved C10 158.8 mm to (49.6, 14.8), flipped to the bottom, turned to 270 degrees
- moved C5 138.8 mm to (18.6, 5.35), flipped to the bottom, turned to 180 degrees
- moved C9 137.5 mm to (48.0, 14.9), flipped to the bottom, turned to 270 degrees
- moved R14 136.2 mm to (18.4, 17.7), flipped to the bottom, turned to 180 degrees
- moved R4 130.5 mm to (12.4, 5.25), flipped to the bottom
- moved R12 130.1 mm to (18.5, 15.6), flipped to the bottom
- moved C15 128.7 mm to (27.3, 18.5), flipped to the bottom, turned to 90 degrees
- moved R13 128.6 mm to (18.5, 7.09), flipped to the bottom, turned to 180 degrees
- moved C1 125.6 mm to (8.83, 32.5), flipped to the bottom, turned to 270 degrees
- moved R31 120.2 mm to (25.5, 18.4), flipped to the bottom, turned to 270 degrees
- moved R1 119.9 mm to (32.2, 15.7), flipped to the bottom, turned to 270 degrees
- moved R11 119.1 mm to (18.5, 11.4), flipped to the bottom
- moved C14 117.0 mm to (23.8, 18.4), flipped to the bottom, turned to 90 degrees
- moved C4 112.7 mm to (21.4, 32.4), flipped to the bottom, turned to 270 degrees
- moved D1 110.0 mm to (7.27, 32.0), flipped to the bottom, turned to 270 degrees
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Connections:
- removed net +4.1V: C10.1, C12.1, C13.1, C8.1, C9.1, D2.2, D3.2, IC1.6, IC1.7, R1.1, R11.1, R12.1, R21.1, R22.1, R29.2, R30.1, R31.1, U3.8, U4.2
- net 3.3V: now also C10.1, C12.1, C13.1, C8.1, C9.1, D2.2, D3.2, IC1.6, IC1.7, R1.1, R11.1, R12.1, R21.1, R22.1, R29.2, R30.1, R31.1, U3.8, U4.2
- net ADC_ALERT: now also U4.31
- net ADC_SCL: now also U4.36
- net ADC_SDA: now also U4.33
- net BUTTON_PROG: now also U4.37
- net IO0: now also U4.25
- net LED_BLUE: now also U4.12
- net LED_GREEN: now also U4.11
- net LED_RED: now also U4.10
Routing:
- net 3.3V: track 0.00 -> 206.3 mm, vias 0 -> 7
- net ADC_VOLTAGE_L2: track 0.00 -> 120.7 mm
- net NEUTRAL: track 0.00 -> 91.7 mm, vias 0 -> 1
- net L1_VOLTAGE: track 0.00 -> 63.8 mm, vias 0 -> 1
- net IO0: track 0.00 -> 59.4 mm, vias 0 -> 4
- net ADC_VOLTAGE_L1: track 0.00 -> 58.7 mm, vias 0 -> 2
- net PE: track 0.00 -> 58.5 mm
- net L2_VOLTAGE: track 0.00 -> 57.1 mm
- net ADC_CURRENT_L1: track 0.00 -> 54.9 mm, vias 0 -> 2
- net 5V: track 0.00 -> 54.8 mm, vias 0 -> 2
- net BUTTON_PROG: track 0.00 -> 51.1 mm, vias 0 -> 2
- net LED_GREEN: track 0.00 -> 50.0 mm, vias 0 -> 2
- net ADC_SCL: track 0.00 -> 47.1 mm
- net ADC_SDA: track 0.00 -> 38.4 mm
- net ADC_CURRENT_L2: track 0.00 -> 36.3 mm, vias 0 -> 2
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- added copper zone on layer 1, net GND
- added copper zone on layer 16, net GND
Other:
- board size 55 x 80 mm -> 55.5 x 70.5 mm

Commit message: PCB layout finished
Parts:
- moved X2 0.77 mm to (3.00, 21.1)
- moved X1 0.67 mm to (3.00, 13.3)
- moved P1 0.34 mm to (12.0, 64.7)
Routing:
- net GND: track 18.6 -> 13.8 mm, vias 144 -> 147
- net LED_GREEN: track 50.0 -> 51.9 mm
- net ADC_CURRENT_L2: track 36.3 -> 37.7 mm
- net LED_RED: track 33.4 -> 34.5 mm
- net 3.3V: track 206.3 -> 207.0 mm
- net N$11: track 20.0 -> 20.6 mm
- net NEUTRAL: track 91.7 -> 91.1 mm
- net ADC_CURRENT_L1: track 54.9 -> 55.5 mm
Other:
- board text added: "PowerSpy"
