File: Hardware/0. Project/PowerSpy.sch (EAGLE design)
At the start: 91 parts, among them IC1 LM324D, IC2 CP2102N-A01-GQFN28, P1 Mini-Fit 4T, T1 SS8050, T2 SS8050, U1 ADS1115IDGST, U2 HLK-PM01, U3 NCP1117ST33T3G, U4 ESP32-WROOM-32D, X1 USB Micro B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

Commit message: Another new and better AFE approach
Parts:
- removed IC1: LM324D, linear:LM324D
- removed R10, R11: 100k (1%), rcl:R-EU_R0603
- removed R13, R34, R35: 10k (1%), rcl:R-EU_R0603
- removed R28, R7: 1M (5%), rcl:R-EU_R0603
- added R50: 47R (5%), rcl:R-EU_R0603
- added U5: MCP6024, MCP6024:MCP6024
- added U6: MCP6021, MCP6024:MCP6021
- C4, C9: value 10uF/10V (20%) -> 10nF/50V (10%)
- R12: value 10k (1%) -> 47R (5%)
- R14, R15: value 100k (1%) -> 200k (1%)
- R17, R18: value 1k6 (1%) -> 1k5 (1%)
- R27: value 47R (5%) -> 100R (5%)
- R5, R6, R8, R9: value 220k (1%) -> 200k (1%)
- X2, X3: value 1503_07 -> Jack J2 Stereo
Connections:
- removed net N$28: R11.2, R15.1
- new net N$35: U5C.+IN, X2.1
- new net N$36: U5D.+IN, X3.1
- new net PE: X2.2
- net +4.1V: now also U5G$1.V+, U6G$2.V+; no longer IC1P.V+
- net 3.3V: no longer R12.1, R34.1
- net ADC_CURRENT_L1: now also C4.1, R12.1; no longer R7.1, X2.1
- net ADC_CURRENT_L2: now also C9.1, R50.1; no longer R28.1, X3.1
- net GND: now also U5G$1.V-, U6G$2.V-; no longer IC1P.V-, R13.2, R28.2, R35.2, R7.2
- net N$11: now also U5C.-IN, U5C.OUT; no longer C4.1, R13.1, X2.2
- net N$12: now also R14.1; no longer R10.1
- net N$13: now also U6A.-IN, U6A.OUT; no longer IC1A.-IN, IC1A.OUT
- net N$14: now also U6A.+IN; no longer IC1A.+IN
- net N$15: now also U5A.OUT; no longer IC1B.OUT
- net N$18: now also P1-4.P, R47.2, R48.2, R49.2; no longer R10.2, R14.1
- net N$20: now also U5B.OUT; no longer IC1C.OUT
- net N$22: now also R50.2, U5D.-IN, U5D.OUT; no longer C9.1, R34.2, R35.1, X3.2
- net N$27: now also R15.1; no longer R11.1
- net N$30: now also U5A.-IN; no longer IC1B.-IN
- net N$32: now also U5A.+IN; no longer IC1B.+IN
- net N$33: now also U5B.-IN; no longer IC1C.-IN
- net N$34: now also U5B.+IN; no longer IC1C.+IN
- net NEUTRAL: now also X3.2; no longer R47.2, R48.2, R49.2
Other:
- note added: "AC/DC Converter Module 3W / 5V"
- note added: "Máx. 1,65V"
- note removed: "AC/DC Converter Module"
- moved on the sheet: C1, C11, C12, C15, C17, C18, C2, C4, C5, C6, C7, C8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

Commit message: Schematic parts renumbered
Parts:
- removed R44: S05K230, varistor:VARISTORS05K11
- removed R45, R46, R47, R48, R49: S05K130, varistor:VARISTORS05K11
- added R10, R11, R7: 200k (1%), rcl:R-EU_R0603
- added R13: 1k5 (1%), rcl:R-EU_R0603
- added R34, R35: 10k (5%), rcl:R-EU_R0603
- C4: value 10nF/50V (10%) -> 4.7uF/6.3V (10%)
- C5: value 4.7uF/6.3V (10%) -> 10nF/50V (10%)
- R12: value 47R (5%) -> 1k5 (1%)
- R14, R15: value 200k (1%) -> 220R (5%)
- R16, R19: value 220R (5%) -> 100k (1%)
- R17: value 1k5 (1%) -> 220R (5%)
- R18: value 1k5 (1%) -> 100k (1%)
- R21: value 220R (5%) -> 10k (5%)
- R22: value 100k (1%) -> 100R (5%)
- R23: value 100k (1%) -> 47R (5%)
- R24: value 100k (1%) -> 2k (5%)
- R25: value 10k (5%) -> 10k (5%)(NC)
- R26: value 47R (5%) -> 0R (5%)
- R27: value 100R (5%) -> 0R (5%)
- R29: value 2k (5%) -> 150R (5%)
- R30: value 10k (5%)(NC) -> 50R (5%)
- R31: value 0R (5%) -> 10k (5%)
- R32: value 0R (5%) -> 50R (5%)
- R33: value 150R (5%) -> 10k (5%)
- R36, R37: value 50R (5%) -> 10k (5%)
- R38: value 10k (5%) -> S05K230; device rcl:R-EU_R0603 -> varistor:VARISTORS05K11
- R39, R40, R41, R42, R43: value 10k (5%) -> S05K130; device rcl:R-EU_R0603 -> varistor:VARISTORS05K11
- R9: value 200k (1%) -> 47R (5%)
- U1: value ADS1115IDGST -> MCP6021; device ADS1115IDGST:ADS1115IDGST -> MCP6024:MCP6021
- U2: value HLK-PM01 -> MCP6024; device HLK-PM01:HLK-PM01 -> MCP6024:MCP6024
- U3: value NCP1117ST33T3G -> ADS1115IDGST; device REG1117:REG1117 -> ADS1115IDGST:ADS1115IDGST
- U4: value ESP32-WROOM-32D -> HLK-PM01; device ESP32-WROOM-32D:ESP32-WROOM-32D -> HLK-PM01:HLK-PM01
- U5: value MCP6024 -> NCP1117ST33T3G; device MCP6024:MCP6024 -> REG1117:REG1117
- U6: value MCP6021 -> ESP32-WROOM-32D; device MCP6024:MCP6021 -> ESP32-WROOM-32D:ESP32-WROOM-32D
- renumbered IC2 to IC1, P1 to CN1, R50 to R28
Connections:
- net +4.1V: now also U1G$2.V+, U2G$1.V+; no longer U5G$1.V+, U6G$2.V+
- net 3.3V: now also C4.1, R21.1, R24.2, R34.1, R35.1, R36.1, R37.1, U3.VDD, U5.VOUT, U6.3V3; no longer C5.1, R25.1, R29.2, R40.1, R41.1, R42.1, R43.1, U1.VDD, U3.VOUT, U4.3V3
- net 5V: now also U5.VIN; no longer U3.VIN
- net ADC_ALERT: now also U3.ALERT/RDY, U6.IO19; no longer U1.ALERT/RDY, U4.IO19
- net ADC_CURRENT_L1: now also C5.1, R9.1, U3.AIN0, U6.IO32; no longer C4.1, R12.1, U1.AIN0, U4.IO32
- net ADC_CURRENT_L2: now also U3.AIN2, U6.IO33; no longer U1.AIN2, U4.IO33
- net ADC_SCL: now also R35.2, U3.SCL, U6.IO22; no longer R41.2, U1.SCL, U4.IO22
- net ADC_SDA: now also R37.2, U3.SDA, U6.IO21; no longer R42.2, U1.SDA, U4.IO21
- net ADC_VOLTAGE_L1: now also R23.1, U3.AIN1, U6.IO34; no longer R26.1, U1.AIN1, U4.IO34
- net ADC_VOLTAGE_L2: now also R22.1, U3.AIN3, U6.IO35; no longer R27.1, U1.AIN3, U4.IO35
- net BUTTON_PROG: now also R21.2, U6.IO23; no longer R25.2, U4.IO23
- net DTR: now also R31.2; no longer R38.2
- net EN: now also R36.2, U6.EN; no longer R43.2, U4.EN
- net GND: now also R25.1, U1G$2.V-, U2G$1.V-, U3.ADDR, U4.VO-, U5.GND, U6.GND; no longer R30.1, U1.ADDR, U1.GND, U2.VO-, U4.GND, U5G$1.V-, U6G$2.V-
- net IO0: now also R34.2, U6.IO0; no longer R40.2, U4.IO0
- net L1_VOLTAGE: now also R38.1, R39.1, R43.1, R6.1, U4.AC1; no longer R44.1, R45.1, R49.1, R5.1, U2.AC1
- net L2_VOLTAGE: now also R38.2, R40.1, R42.1, R5.1; no longer R44.2, R46.1, R48.1, R6.1
- net LED_BLUE: now also R32.1, U6.IO27; no longer R37.1, U4.IO27
- net LED_GREEN: now also R30.1, U6.IO26; no longer R36.1, U4.IO26
- net LED_RED: now also R29.1, U6.IO25; no longer R33.1, U4.IO25
- net N$1: now also R25.2; no longer R30.2
- net N$10: now also R27.2; no longer R32.2
- net N$11: now also R9.2, U2C.-IN, U2C.OUT; no longer R12.2, U5C.-IN, U5C.OUT
- net N$12: now also R11.1; no longer R14.1
- net N$13: now also R14.2, U1A.-IN, U1A.OUT; no longer R16.2, U6A.-IN, U6A.OUT
- net N$14: now also U1A.+IN; no longer U6A.+IN
- net N$15: now also R19.1, R23.2, U2A.OUT; no longer R23.1, R26.2, U5A.OUT
- net N$16: now also R10.2, R12.1; no longer R18.1, R19.2
- net N$18: now also R41.2, R42.2, R43.2; no longer R47.2, R48.2, R49.2
- net N$19: now also R6.2; no longer R5.2
- net N$2: now also R24.1; no longer R29.1
- net N$20: now also R20.1, R22.2, U2B.OUT; no longer R24.1, R27.2, U5B.OUT
- net N$21: now also R30.2; no longer R36.2
- net N$22: now also U2D.-IN, U2D.OUT; no longer U5D.-IN, U5D.OUT
- net N$26: now also R32.2; no longer R37.2
- net N$27: now also R10.1, R7.2; no longer R15.1, R9.2
- net N$29: now also R5.2, R7.1; no longer R6.2, R9.1
- net N$3: now also R29.2; no longer R33.2
- net N$30: now also R18.1, R19.2, U2A.-IN; no longer R22.1, R23.2, U5A.-IN
- net N$31: now also R11.2, R13.1, R17.2; no longer R14.2, R17.1, R21.2
- net N$32: now also R17.1, U2A.+IN; no longer R21.1, U5A.+IN
- net N$33: now also R16.1, R20.2, U2B.-IN; no longer R20.1, R24.2, U5B.-IN
- net N$34: now also R15.1, U2B.+IN; no longer R19.1, U5B.+IN
- net N$35: now also U2C.+IN; no longer U5C.+IN
- net N$36: now also U2D.+IN; no longer U5D.+IN
- net N$5: now also R33.1; no longer R39.1
- net N$6: now also U4.VO+; no longer U2.VO+
- net N$7: now also R31.1; no longer R38.1
- net N$8: now also R26.2; no longer R31.2
- net NEUTRAL: now also R12.2, R13.2, R14.1, R16.2, R39.2, R40.2, R41.1, U4.AC2; no longer R16.1, R17.2, R20.2, R22.2, R45.2, R46.2, R47.1, U2.AC2
- net RTS: now also R33.2; no longer R39.2
- net USB_RX: now also R27.1, U6.TXD0; no longer R32.1, U4.TXD0
- net USB_TX: now also R26.1, U6.RXD0; no longer R31.1, U4.RXD0
Other:
- moved on the sheet: C4, C5, R12, R14, R15, R16, R17, R18, R19, R20, R21, R22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

Commit message: Minor improvements
Parts:
- added C19: 100nF/50V (10%), rcl:C-EUC0603K
- C3: value 10uF/10V (20%) -> 100nF/50V (10%)
Connections:
- net +4.1V: now also C19.1
- net GND: now also C19.2
Other:
- moved on the sheet: C5, C9, R28, R9, U2C, U2D, X2, X3

Commit message: ADS1115 7-bits slave address added to schematic
Other:
- note added: "7-bits Slave Address 0b1001000 0x48"
Changed lines of the file:
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@@
 <text x="22.86" y="167.64" size="1.778" layer="97">Máx. 1,65V</text>
 <text x="120.65" y="167.64" size="1.778" layer="97">Máx. 1,65V</text>
+<text x="215.9" y="75.565" size="1.778" layer="97" font="vector" align="center">7-bits Slave Address
+0b1001000
+0x48</text>
 </plain>
 <instances>

Commit message: Pull-down resistor added to current AFE
Parts:
- added R44, R45: 1M (5%), rcl:R-EU_R0603
Connections:
- net GND: now also R44.2, R45.2
- net N$35: now also R44.1
- net N$36: now also R45.1
Other:
- note added: "Vp-max 1,65V"
- note removed: "Máx. 1,65V"
- moved on the sheet: X2
Changed lines of the file:
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@@
 <part name="C19" library="rcl" library_urn="urn:adsk.eagle:library:334" deviceset="C-EU" device="C0603K" package3d_urn="urn:adsk.eagle:package:23680/2" value="100nF/50V (10%)"/>
 <part name="GND9" library="supply1" library_urn="urn:adsk.eagle:library:371" deviceset="GND" device=""/>
+<part name="R44" library="rcl" library_urn="urn:adsk.eagle:library:334" deviceset="R-EU_" device="R0603" package3d_urn="urn:adsk.eagle:package:23555/3" value="1M (5%)"/>
+<part name="GND10" library="supply1" library_urn="urn:adsk.eagle:library:371" deviceset="GND" device=""/>
+<part name="R45" library="rcl" library_urn="urn:adsk.eagle:library:334" deviceset="R-EU_" device="R0603" package3d_urn="urn:adsk.eagle:package:23555/3" value="1M (5%)"/>
+<part name="GND16" library="supply1" library_urn="urn:adsk.eagle:library:371" deviceset="GND" device=""/>
 </parts>
 <sheets>
@@
 <text x="5.715" y="253.365" size="2.54" layer="152">VIRTUAL GROUND REFERENCE</text>
 <wire x1="4.445" y1="196.85" x2="107.315" y2="196.85" width="0.254" layer="152" style="longdash"/>
-<text x="22.86" y="167.64" size="1.778" layer="97">Máx. 1,65V</text>
-<text x="120.65" y="167.64" size="1.778" layer="97">Máx. 1,65V</text>
+<text x="28.702" y="173.863" size="1.4224" layer="97" font="vector" align="center">Vp-max
+1,65V</text>
 <text x="215.9" y="75.565" size="1.778" layer="97" font="vector" align="center">7-bits Slave Address
 0b1001000
 0x48</text>
+<text x="127.762" y="173.863" size="1.4224" layer="97" font="vector" align="center">Vp-max
+1,65V</text>
+<text x="78.232" y="98.298" size="1.4224" layer="97" font="vector" align="center">Vp-max
+1,65V</text>
+<text x="79.502" y="137.668" size="1.4224" layer="97" font="vector" align="center">Vp-max
+1,65V</text>
 </plain>
 <instances>
@@
 <attribute name="VALUE" x="224.79" y="59.69" size="1.778" layer="96"/>
 </instance>
-<instance part="X2" gate="G$1" x="15.24" y="165.1" smashed="yes" rot="R180">
-<attribute name="NAME" x="8.255" y="176.149" size="1.778" layer="95"/>
-<attribute name="VALUE" x="8.255" y="173.99" size="1.778" layer="96"/>
+<instance part="X2" gate="G$1" x="13.97" y="165.1" smashed="yes" rot="R180">
+<attribute name="NAME" x="6.604" y="169.164" size="1.778" layer="95"/>
+<attribute name="VALUE" x="6.985" y="159.385" size="1.4224" layer="96"/>
 </instance>
 <instance part="U3" gate="A" x="215.9" y="103.505" smashed="yes">
@@
 </instance>
 <instance part="X3" gate="G$1" x="113.03" y="165.1" smashed="yes" rot="R180">
-<attribute name="NAME" x="106.68" y="176.149" size="1.778" layer="95"/>
-<attribute name="VALUE" x="106.68" y="173.99" size="1.778" layer="96"/>
+<attribute name="NAME" x="105.918" y="168.529" size="1.778" layer="95"/>
+<attribute name="VALUE" x="106.045" y="160.02" size="1.4224" layer="96"/>
 </instance>
 <instance part="R22" gate="G$1" x="124.46" y="92.075" smashed="yes" rot="MR0">
@@
 <instance part="GND9" gate="1" x="61.595" y="173.355" smashed="yes">
 <attribute name="VALUE" x="59.055" y="170.815" size="1.778" layer="96"/>
+</instance>
+<instance part="R44" gate="G$1" x="29.21" y="161.29" smashed="yes" rot="MR270">
+<attribute name="NAME" x="27.5209" y="158.75" size="1.27" layer="95" rot="R90"/>
+<attribute name="VALUE" x="30.861" y="157.734" size="1.27" layer="96" rot="MR90"/>
+</instance>
+<instance part="GND10" gate="1" x="29.21" y="150.495" smashed="yes">
+<attribute name="VALUE" x="26.67" y="147.955" size="1.778" layer="96"/>
+</instance>
+<instance part="R45" gate="G$1" x="128.27" y="161.29" smashed="yes" rot="MR270">
+<attribute name="NAME" x="126.5809" y="158.75" size="1.27" layer="95" rot="R90"/>
+<attribute name="VALUE" x="129.921" y="157.734" size="1.27" layer="96" rot="MR90"/>
+</instance>
+<instance part="GND16" gate="1" x="128.27" y="150.495" smashed="yes">
+<attribute name="VALUE" x="125.73" y="147.955" size="1.778" layer="96"/>
 </instance>
 </instances>
@@
 <wire x1="61.595" y1="177.165" x2="58.42" y2="177.165" width="0.1524" layer="91"/>
 </segment>
+<segment>
+<pinref part="GND10" gate="1" pin="GND"/>
+<pinref part="R44" gate="G$1" pin="2"/>
+<wire x1="29.21" y1="153.035" x2="29.21" y2="156.21" width="0.1524" layer="91"/>
+</segment>
+<segment>
+<pinref part="GND16" gate="1" pin="GND"/>
+<pinref part="R45" gate="G$1" pin="2"/>
+<wire x1="128.27" y1="153.035" x2="128.27" y2="156.21" width="0.1524" layer="91"/>
+</segment>
 </net>
 <net name="3.3V" class="0">
@@
 <pinref part="U2" gate="C" pin="+IN"/>
 <pinref part="X2" gate="G$1" pin="1"/>
-<wire x1="38.1" y1="170.18" x2="20.32" y2="170.18" width="0.1524" layer="91"/>
+<wire x1="38.1" y1="170.18" x2="29.21" y2="170.18" width="0.1524" layer="91"/>
+<pinref part="R44" gate="G$1" pin="1"/>
+<wire x1="29.21" y1="170.18" x2="19.05" y2="170.18" width="0.1524" layer="91"/>
+<wire x1="29.21" y1="166.37" x2="29.21" y2="170.18" width="0.1524" layer="91"/>
+<junction x="29.21" y="170.18"/>
 </segment>
 </net>
@@
 <pinref part="X3" gate="G$1" pin="1"/>
 <pinref part="U2" gate="D" pin="+IN"/>
-<wire x1="118.11" y1="170.18" x2="136.525" y2="170.18" width="0.1524" layer="91"/>
+<wire x1="118.11" y1="170.18" x2="128.27" y2="170.18" width="0.1524" layer="91"/>
+<pinref part="R45" gate="G$1" pin="1"/>
+<wire x1="128.27" y1="170.18" x2="136.525" y2="170.18" width="0.1524" layer="91"/>
+<wire x1="128.27" y1="166.37" x2="128.27" y2="170.18" width="0.1524" layer="91"/>
+<junction x="128.27" y="170.18"/>
 </segment>
 </net>
@@
 <segment>
 <pinref part="X2" gate="G$1" pin="2"/>
-<wire x1="20.32" y1="162.56" x2="21.59" y2="162.56" width="0.1524" layer="91"/>
+<wire x1="19.05" y1="162.56" x2="21.59" y2="162.56" width="0.1524" layer="91"/>
 <wire x1="21.59" y1="162.56" x2="21.59" y2="153.67" width="0.1524" layer="91"/>
 <pinref part="PE4" gate="M" pin="PE"/>

Commit message: ESP32 JLINK Pins added
Connections:
- new net JLINK-TCK: U6.IO13
- new net JLINK-TDI: U6.IO12
- new net JLINK-TDO: U6.IO15
- new net JLINK-TMS: U6.IO14
Other:
- note added: "2.1"
- note removed: "2.0"
Changed lines of the file:
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@@
 <text x="307.975" y="26.035" size="3.81" layer="94">Tiago Silva</text>
 <text x="290.83" y="19.685" size="2.54" layer="94">github.com/TiagoPaulaSilva/PowerSpy</text>
-<text x="377.825" y="1.27" size="2.54" layer="94" ratio="5">2.0</text>
+<text x="377.825" y="1.27" size="2.54" layer="94" ratio="5">2.1</text>
 <text x="306.705" y="6.35" size="2.54" layer="94" ratio="5">Complete Schematic</text>
 <text x="261.62" y="154.94" size="1.778" layer="97" align="center">AC/DC Converter Module
@@
 </segment>
 </net>
+<net name="JLINK-TDO" class="0">
+<segment>
+<pinref part="U6" gate="G$1" pin="IO15"/>
+<wire x1="358.14" y1="90.17" x2="361.95" y2="90.17" width="0.1524" layer="91"/>
+<label x="361.95" y="90.17" size="1.27" layer="95" xref="yes"/>
+</segment>
+</net>
+<net name="JLINK-TCK" class="0">
+<segment>
+<pinref part="U6" gate="G$1" pin="IO13"/>
+<wire x1="358.14" y1="95.25" x2="361.95" y2="95.25" width="0.1524" layer="91"/>
+<label x="361.95" y="95.25" size="1.27" layer="95" xref="yes"/>
+</segment>
+</net>
+<net name="JLINK-TDI" class="0">
+<segment>
+<pinref part="U6" gate="G$1" pin="IO12"/>
+<wire x1="358.14" y1="97.79" x2="361.95" y2="97.79" width="0.1524" layer="91"/>
+<label x="361.95" y="97.79" size="1.27" layer="95" xref="yes"/>
+</segment>
+</net>
+<net name="JLINK-TMS" class="0">
+<segment>
+<pinref part="U6" gate="G$1" pin="IO14"/>
+<wire x1="358.14" y1="92.71" x2="361.95" y2="92.71" width="0.1524" layer="91"/>
+<label x="361.95" y="92.71" size="1.27" layer="95" xref="yes"/>
+</segment>
+</net>
